File: KiCad/RTC8088.kicad_sch (KiCad schematic)
At the start: 9 parts, among them SW1 Address Select, U1 DS12885, U2 ATF16V8B, Y1 32768Hz

Commit message: Replace tht DS12855 with smt bq3285
Parts:
- added C2: 0.1uF, Capacitor_THT:C_Disc_D4.7mm_W2.5mm_P5.00mm, symbol Device:C
- C1: footprint My_Components:Cap_Cer_508 -> Capacitor_THT:C_Disc_D4.7mm_W2.5mm_P5.00mm
- U1: value DS12885 -> BQ3285; footprint My_Components:IC_DIP24_600 -> Package_SO:SOIC-24W_7.5x15.4mm_P1.27mm
Connections:
- net GND: now also C2.2
- net VCC: now also C2.1
- net at U1.2 (X1): now also Y1.2; no longer Y1.1
- net at U1.3 (X2): now also Y1.1; no longer Y1.2
Other:
- company: Sergey Kiselev -> [zyga64]
- moved on the sheet: C1
